File: QCW_Bridge/QCW_Bridge.kicad_pcb (KiCad board)
At the start: 2 copper layers, 501.5 x 295.5 mm, 11 parts, among them J1 Conn_01x01, J2 Conn_01x01, J3 Conn_01x01, J4 Conn_01x01, J5 Conn_01x01, Q1 SiCFET_LeadBent, Q2 SiCFET_LeadBent, Q3 SiCFET_LeadBent, Q4 SiCFET_LeadBent

Commit message: update bridge
Parts:
- removed C1: 25u film, Project:EZPV1B256MTB
- removed J2, J5: Conn_01x01, Project:M6 Lug
- removed Q3, Q4: SiCFET_LeadBent, Project:PG-TO247 Bent
- J1, J3, J4: footprint Project:M6 Lug -> Project:WirePad_8AWG
- moved J3 331.8 mm to (303.5, 226.7)
- moved J4 327.9 mm to (361.9, 216.5)
- moved C13 292.3 mm to (332.7, 231.8)
- moved Q2 292.1 mm to (348.0, 209.6)
- moved Q1 289.8 mm to (322.6, 209.6)
- moved J1 237.7 mm to (332.7, 226.7), turned to 180 degrees
Routing:
- added copper zone on B.Cu, net Net-(J4-Pin_1)
- removed copper zone on F.Cu, net Net-(J5-Pin_1)
Other:
- board size 501.5 x 295.5 mm -> 76.2 x 44.4 mm
