File: QCW_Bridge/QCW_Bridge.kicad_sch (KiCad schematic)
At the start: 11 parts, among them J1 Conn_01x01, J2 Conn_01x01, J3 Conn_01x01, J4 Conn_01x01, J5 Conn_01x01, Q1 SiCFET_LeadBent, Q2 SiCFET_LeadBent, Q3 SiCFET_LeadBent, Q4 SiCFET_LeadBent

Commit message: update bridge
Parts:
- removed C1: 25u film, Project:EZPV1B256MTB, symbol Device:C
- removed J2, J5: Conn_01x01, Project:M6 Lug, symbol Connector_Generic:Conn_01x01
- removed Q3, Q4: SiCFET_LeadBent, Project:PG-TO247 Bent, symbol Project:SiCFET_LeadBent
- J1, J3, J4: footprint Project:M6 Lug -> Project:WirePad_8AWG
