File: QCW_Link/QCW_Link.kicad_pcb (KiCad board)
At the start: 2 copper layers, 420 x 180 mm, 19 parts, among them J1 Conn_01x01, J2 Conn_01x01, J3 Conn_01x01, J4 Conn_01x01, J5 Conn_01x01, J6 Conn_01x01, J7 Conn_01x01

Commit message: update bridge
Parts:
- J6, J7: moved to F.Cu
- moved J5 275.2 mm to (208.0, -8.00)
- moved J1 265.0 mm to (165.0, 188.0)
- moved J6 227.7 mm to (174.0, 204.0)
- moved J4 213.8 mm to (180.0, -8.00)
- moved C2 201.2 mm to (225.0, 45.0), turned to 90 degrees
- moved C4 201.2 mm to (315.0, 45.0), turned to 90 degrees
- moved C5 201.2 mm to (45.0, 135.0)
- moved C7 201.2 mm to (135.0, 135.0)
- moved R8 188.5 mm to (270.0, 162.9), turned to 90 degrees
- moved J7 180.7 mm to (185.0, 204.0)
- moved R5 180.0 mm to (90.0, 17.1)
- moved J2 177.2 mm to (195.0, 188.0)
- moved J3 164.4 mm to (152.0, -8.00)
- moved R7 90.0 mm to (90.0, 107.1)
- moved R6 34.1 mm to (270.0, 72.9), turned to 90 degrees
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Routing:
- removed copper zone on B.Cu, net Net-(J1-Pin_1)
- removed copper zone on B.Cu, net Net-(J2-Pin_1)
- removed copper zone on F.Cu, net Net-(J4-Pin_1)
Other:
- board size 420 x 180 mm -> 380 x 236 mm
